Commit message: camera, ik and move_base now are working fine

File: urdf/my_robot.xacro (robot description, xacro)
@@ -1,5 +1,5 @@
 <?xml version="1.0"?>
 <robot xmlns:xacro="http://www.ros.org/wiki/xacro" name="robot2_laser_xacro">
-<xacro:include filename="$(find assignment2)/urdf/robot2_laser.gazebo"/>
+<xacro:include filename="$(find assignment2)/urdf/my_robot.gazebo"/>
 	<xacro:property name="length_wheel" value="0.02" />
 	<xacro:property name="radius_wheel" value="0.05" />
@@ -150,5 +150,5 @@
 		<origin xyz="0 0 0" rpy="0 0 0"/>
 		<geometry>
-			<cylinder radius="0.02" length="0.04"/>
+			<cylinder radius="0.02" length="0.16"/>
 		</geometry>
 	</collision>
@@ -156,5 +156,5 @@
 		<origin xyz="0 0 0" rpy="0 0 0"/>
 		<geometry>
-			<cylinder radius="0.02" length="0.04"/>
+			<cylinder radius="0.02" length="0.16"/>
 		</geometry>
 		<material name="red" />
@@ -164,88 +164,7 @@
 	<axis xyz="0 0 1"/>
 	<limit effort="1000.0" lower="-3.14" upper="3.14" velocity="0.2"/>
-	<origin rpy="0 0 0" xyz="0 0 0.045"/>
+	<origin rpy="0 0 0" xyz="0 0 0.1025"/>
 	<parent link="arm_base_link"/>
 	<child link="arm_link_01"/>
-</joint>
-<link name="arm_link_02">
-	<inertial>
-		<mass value="0.00625"/>
-		<origin xyz="0 0 0" rpy="0 0 0" />
-		<inertia ixx="0.00000256975" ixy="0" ixz="0" iyy="0.00000256975" iyz="0" izz="0.00000180625"/>
-	</inertial>
-	<collision>
-		<origin xyz="0 0 0.02" rpy="0 0 0"/>
-		<geometry>
-			<cylinder radius="0.02" length="0.04"/>
-		</geometry>
-	</collision>
-	<visual>
-		<origin xyz="0 0 0.02" rpy="0 0 0"/>
-		<geometry>
-			<cylinder radius="0.02" length="0.04"/>
-		</geometry>
-		<material name="red" />
-	</visual>
-</link>
-<joint name="arm_joint_02" type="revolute">
-	<axis xyz="1 0 0"/>
-	<limit effort="1000.0" lower="-1.8" upper="1.8" velocity="0.2"/>
-	<origin rpy="0 0 0" xyz="0 0 0.02"/>
-	<parent link="arm_link_01"/>
-	<child link="arm_link_02"/>
-</joint>
-<link name="arm_link_03">
-	<inertial>
-		<mass value="0.00625"/>
-		<origin xyz="0 0 0" rpy="0 0 0" />
-		<inertia ixx="0.00000256975" ixy="0" ixz="0" iyy="0.00000256975" iyz="0" izz="0.00000180625"/>
-	</inertial>
-	<collision>
-		<origin xyz="0 0 0.02" rpy="0 0 0"/>
-		<geometry>
-			<cylinder radius="0.02" length="0.04"/>
-		</geometry>
-	</collision>
-	<visual>
-		<origin xyz="0 0 0.02" rpy="0 0 0"/>
-		<geometry>
-			<cylinder radius="0.02" length="0.04"/>
-		</geometry>
-		<material name="red" />
-	</visual>
-</link>
-<joint name="arm_joint_03" type="revolute">
-	<axis xyz="1 0 0"/>
-	<limit effort="1000.0" lower="-1.8" upper="1.8" velocity="0.2"/>
-	<origin rpy="0 0 0" xyz="0 0 0.04"/>
-	<parent link="arm_link_02"/>
-	<child link="arm_link_03"/>
-</joint>
-<link name="arm_link_04">
-	<inertial>
-		<mass value="0.00625"/>
-		<origin xyz="0 0 0" rpy="0 0 0" />
-		<inertia ixx="0.00000256975" ixy="0" ixz="0" iyy="0.00000256975" iyz="0" izz="0.00000180625"/>
-	</inertial>
-	<collision>
-		<origin xyz="0 0 0.02" rpy="0 0 0.785"/>
-		<geometry>
-			<box size="0.017 0.1 0.04"/>
-		</geometry>
-	</collision>
-	<visual>
-		<origin xyz="0 0 0.02" rpy="0 0 0.785"/>
-		<geometry>
-			<box size="0.017 0.1 0.04"/>
-		</geometry>
-		<material name="red" />
-	</visual>
-</link>
-<joint name="arm_joint_04" type="revolute">
-	<axis xyz="1 0 0"/>
-	<limit effort="1000.0" lower="-1.8" upper="1.8" velocity="0.5"/>
-	<origin rpy="0 0 0" xyz="0 0 0.04"/>
-	<parent link="arm_link_03"/>
-	<child link="arm_link_04"/>
 </joint>
   <link name="hokuyo_link">
@@ -273,5 +192,5 @@
   <joint name="hokuyo_joint" type="fixed">
 	    <axis xyz="0 1 0" />
-	    <origin xyz="0 0 0.15" rpy="0 0 0"/>
+	    <origin xyz="0.14 0 0.025" rpy="0 0 0"/>
 	    <parent link="link_chassis"/>
 	    <child link="hokuyo_link"/>
@@ -279,6 +198,6 @@
   <joint name="camera_joint" type="fixed">
     <axis xyz="0 1 0" />
-    <origin xyz="0 0 0.8" rpy="0 0 0"/>
-    <parent link="arm_link_04"/>
+    <origin xyz="0 0 0.1" rpy="0 0 0"/>
+    <parent link="arm_link_01"/>
     <child link="camera_link"/>
   </joint>
@@ -286,7 +205,7 @@
   <link name="camera_link">
     <collision>
-      <origin xyz="0.05 0.05 0.05" rpy="0 0 0"/>
-      <geometry>
-    <box size="0.05 0.05 0.05"/>
+      <origin xyz="0.0 0.0 0.0" rpy="0 0 0"/>
+      <geometry>
+    <box size="0.02 0.02 0.02"/>
       </geometry>
     </collision>
@@ -294,5 +213,5 @@
       <origin xyz="0 0 0" rpy="0 0 0"/>
       <geometry>
-    <box size="$0.05 0.05 0.05"/>
+    <box size="0.02 0.02 0.02"/>
       </geometry>
       <material name="red"/>

File: urdf/test.urdf (robot description, URDF)
Before this commit: robot robot2_laser_xacro, 10 links, 9 joints
Links:
- removed link arm_link_02
- removed link arm_link_03
- removed link arm_link_04
- link arm_link_01: geometry collision cylinder length=0.16 radius=0.02; visual cylinder length=0.16 radius=0.02
Joints:
- removed joint arm_joint_02
- removed joint arm_joint_03
- removed joint arm_joint_04
- joint arm_joint_01: origin xyz=0 0 0.045 rpy=0 0 0 -> xyz=0 0 0.1025 rpy=0 0 0
- joint camera_joint: origin xyz=0 0 0.08 rpy=0 0 0 -> xyz=0 0 0.1 rpy=0 0 0; parent arm_link_04 -> arm_link_01
